Commit message: Changiing the urdf of panda + softhand

File: robot/panda_softhand.urdf.xacro (robot description, xacro)
@@ -3,16 +3,15 @@
   <!-- MODELS -->
   <xacro:include filename="$(find franka_description)/robots/panda_arm.urdf.xacro"/>
-  <xacro:include filename="$(find soft_hand_description)/model/soft_hand_soma_panda.urdf.xacro"/>
+  <xacro:include filename="$(find soft_hand_description)/model/soft_hand_soma_ocado.urdf.xacro"/>
   <link name="world"/>
   <!-- PANDA ARM -->
-  <xacro:panda_arm name="panda_arm" parent="world">
-    <origin xyz="0.0 0.0 0.0" rpy="0.0 0.0 0.0"/>
+  <xacro:panda_arm>
   </xacro:panda_arm>
   <!-- RIGHT SOFTHAND -->
-  <xacro:soft_hand_soma_panda parent="panda_link8" name="right_hand" left="false" withAdaptiveTransmission="true" useMimicTag="$(arg use_mimic_tag)">
+  <xacro:soft_hand_soma_ocado parent="panda_link8" name="right_hand" left="false" withAdaptiveTransmission="true" useMimicTag="true">
     <origin xyz="0 0 0" rpy="0 0 3.1415"/>
-  </xacro:soft_hand_soma_panda>
+  </xacro:soft_hand_soma_ocado>
   <!-- EXTRA ENDEFFECTOR -->
-  <joint name="right_hand_ee_joint" type="fixed">
+  <!-- <joint name="right_hand_ee_joint" type="fixed">
     <origin xyz="0.002 0.00695 0.1" rpy="0 -1.5708 3.1415"/>
     <parent link="right_hand_panda_flange" />
@@ -20,4 +19,4 @@
   </joint>
   <link name="right_hand_ee_link">
-  </link>
+  </link> -->
 </robot>

Commit message: Now the robot urdf is valid but tuning is needed

File: robot/panda_softhand.urdf.xacro (robot description, xacro)
@@ -1,15 +1,14 @@
-<?xml version="1.0"?>
+<?xml version="1.0" encoding='utf-8'?>
 <robot xmlns:xacro="http://www.ros.org/wiki/xacro" name="panda_softhand">
   <!-- MODELS -->
-  <xacro:include filename="$(find franka_description)/robots/panda_arm.urdf.xacro"/>
-  <xacro:include filename="$(find soft_hand_description)/model/soft_hand_soma_ocado.urdf.xacro"/>
-  <link name="world"/>
+  <xacro:include filename="$(find franka_description)/robots/panda_arm.xacro"/>
+  <xacro:include filename="$(find soft_hand_description)/model/soft_hand_soma_panda.urdf.xacro"/>
+  <!-- <link name="world"/> -->
   <!-- PANDA ARM -->
-  <xacro:panda_arm>
-  </xacro:panda_arm>
+  <xacro:panda_arm />
   <!-- RIGHT SOFTHAND -->
-  <xacro:soft_hand_soma_ocado parent="panda_link8" name="right_hand" left="false" withAdaptiveTransmission="true" useMimicTag="true">
+  <xacro:soft_hand_soma_panda parent="panda_link8" name="right_hand" left="false" withAdaptiveTransmission="true" useMimicTag="true">
     <origin xyz="0 0 0" rpy="0 0 3.1415"/>
-  </xacro:soft_hand_soma_ocado>
+  </xacro:soft_hand_soma_panda>
   <!-- EXTRA ENDEFFECTOR -->
   <!-- <joint name="right_hand_ee_joint" type="fixed">

Commit message: Reverted to official model and added extra endeffector link

File: robot/panda_softhand.urdf.xacro (robot description, xacro)
@@ -5,6 +5,6 @@
   <xacro:arg name="robot_ns" default="panda_arm"/>
   <!-- MODELS -->
-  <!-- <xacro:include filename="$(find franka_description)/robots/panda_arm.xacro"/> -->
-  <xacro:include filename="$(find franka_gazebo)/robots/panda_arm.xacro"/>
+  <xacro:include filename="$(find franka_description)/robots/panda_arm.xacro"/>
+  <!-- <xacro:include filename="$(find franka_gazebo)/robots/panda_arm.xacro"/> -->
   <xacro:include filename="$(find soft_hand_description)/model/soft_hand_soma_panda.urdf.xacro"/>
   <!-- Gazebo Stuff -->
@@ -13,9 +13,9 @@
   <!-- <link name="world"/> -->
   <!-- PANDA ARM -->
-  <!-- <xacro:panda_arm /> -->
-  <xacro:panda_arm connected_to='world'/>
+  <xacro:panda_arm />
   <!-- PANDA GAZEBO -->
+  <!-- <xacro:panda_arm connected_to='world'/>
   <xacro:panda_arm_gazebo arm_id="$(arg arm_id)" robot_ns="$(arg robot_ns)"/>
-  <xacro:panda_arm_transmission arm_id="$(arg arm_id)"/>
+  <xacro:panda_arm_transmission arm_id="$(arg arm_id)"/> -->
   <!-- RIGHT SOFTHAND -->
   <xacro:soft_hand_soma_panda parent="panda_link8" name="right_hand" left="false" withAdaptiveTransmission="true" useMimicTag="true">
@@ -23,10 +23,10 @@
   </xacro:soft_hand_soma_panda>
   <!-- EXTRA ENDEFFECTOR -->
-  <!-- <joint name="right_hand_ee_joint" type="fixed">
-    <origin xyz="0.002 0.00695 0.1" rpy="0 -1.5708 3.1415"/>
-    <parent link="right_hand_panda_flange" />
+  <joint name="right_hand_ee_joint" type="fixed">
+    <origin xyz="0.130 0.000 0.035" rpy="0 0 0"/>
+    <parent link="panda_link8" />
     <child link="right_hand_ee_link" />
   </joint>
   <link name="right_hand_ee_link">
-  </link> -->
+  </link>
 </robot>

Commit message: Added world frame

File: robot/panda_softhand.urdf.xacro (robot description, xacro)
@@ -11,5 +11,11 @@
   <xacro:include filename="$(find franka_gazebo)/robots/panda_arm.gazebo.xacro"/>
   <xacro:include filename="$(find franka_gazebo)/robots/panda_arm.transmission.xacro"/>
-  <!-- <link name="world"/> -->
+  <!-- WORLD -->
+  <link name="world"/>
+  <joint name="world_to_panda_joint" type="fixed">
+    <origin xyz="0 0 0" rpy="0 0 0"/>
+    <parent link="world" />
+    <child link="panda_link0" />
+  </joint>
   <!-- PANDA ARM -->
   <xacro:panda_arm />
